Commit message: rt

File: config/kia_niro_frames.urdf (robot description, URDF)
Before this commit: robot kia_niro_ev, 17 links, 16 joints
Links:
- removed link lidar_1/os_imu
- removed link lidar_1/os_lidar
- removed link lidar_1/os_sensor
- removed link lidar_2/os_imu
- removed link lidar_2/os_lidar
- removed link lidar_2/os_sensor
- added link lidar_side/os_imu
- added link lidar_side/os_lidar
- added link lidar_side/os_sensor
- added link lidar_top/os_imu
- added link lidar_top/os_lidar
- added link lidar_top/os_sensor
Joints:
- removed joint base_link_to_lidar_1_os_sensor
- removed joint base_link_to_lidar_2_os_sensor
- removed joint lidar_1_os_sensor_to_os_imu
- removed joint lidar_1_os_sensor_to_os_lidar
- removed joint lidar_2_os_sensor_to_os_imu
- removed joint lidar_2_os_sensor_to_os_lidar
- added joint base_link_to_lidar_side_os_sensor: type fixed, parent base_link, child lidar_side/os_sensor, origin xyz=-0.579812 -0.820105 0.854643 rpy=0.0 0.0 -0.628322
- added joint base_link_to_lidar_top_os_sensor: type fixed, parent base_link, child lidar_top/os_sensor, origin xyz=0.738882 0.006653 1.912894 rpy=0.053872 0.025846 0.000696
- added joint lidar_side_os_sensor_to_os_imu: type fixed, parent lidar_side/os_sensor, child lidar_side/os_imu, origin xyz=0.006253 -0.011775 0.007645 rpy=0.0 0.0 0.0
- added joint lidar_side_os_sensor_to_os_lidar: type fixed, parent lidar_side/os_sensor, child lidar_side/os_lidar, origin xyz=0.0 0.0 0.03618 rpy=0.0 0.0 3.141593
- added joint lidar_top_os_sensor_to_os_imu: type fixed, parent lidar_top/os_sensor, child lidar_top/os_imu, origin xyz=0.006253 -0.011775 0.007645 rpy=0.0 0.0 0.0
- added joint lidar_top_os_sensor_to_os_lidar: type fixed, parent lidar_top/os_sensor, child lidar_top/os_lidar, origin xyz=0.0 0.0 0.0743 rpy=0.0 0.0 3.141593
